File: kicad/9Vsnap.sch (KiCad schematic (older format))
At the start: 11 parts, among them P1 9V_IN, P2 OUT, U1 LM317EMP

Commit message: Done. Gerbers ready
Parts:
- P1: footprint 9Vsnap:9V_clip -> 9Vsnap:9V_clip_968
Changed lines of the file:
@@
 F 0 "P1" H 3000 2700 50  0000 C CNN
 F 1 "9V_IN" V 3100 2550 50  0000 C CNN
-F 2 "9Vsnap:9V_clip" H 3000 2550 60  0001 C CNN
+F 2 "9Vsnap:9V_clip_968" H 3000 2550 60  0001 C CNN
 F 3 "" H 3000 2550 60  0000 C CNN
 	1    3000 2550
